File: Keyboard-PCB-Tutorial.kicad_sch (KiCad schematic)
At the start: 0 parts

Commit message: Create most of the schematic
Parts:
- added C1: 4.7uF, symbol Device:C
- added C2, C4, C5: 0.1uF, symbol Device:C
- added C3, C6, C7: 1uF, symbol Device:C
- added F1: 1A, symbol Device:Polyfuse
- added J1: USB_C_Receptacle_USB2.0_16P, symbol Connector:USB_C_Receptacle_USB2.0_16P
- added R1: 10k, symbol Device:R
- added R2, R3: 5.1k, symbol Device:R
- added SW1: SW_Push, symbol Switch:SW_Push
- added SW2: SW_SPDT, symbol Switch:SW_SPDT
- added U1: STM32G0B1CBTx, Package_QFP:LQFP-48_7x7mm_P0.5mm, symbol MCU_ST_STM32G0:STM32G0B1CBTx
- added U2: SRV05-4, Package_TO_SOT_SMD:SOT-23-6, symbol Power_Protection:SRV05-4
- added U3: XC6206P332MR, Package_TO_SOT_SMD:SOT-23-3, symbol Regulator_Linear:XC6206PxxxMR
Connections:
- new net: J1.A5 (CC1), R3.1
- new net: J1.B5 (CC2), R2.1
- new net: R1.2, SW2.2 (B)
- new net +3.3V: C1.1, C2.1, C3.1, C4.1, C7.1, SW2.3 (C), U1.4 (VBAT), U1.5 (VREF+), U1.6 (VDD), U3.2 (VO)
- new net +5V: C6.1, F1.2, U2.5 (VP), U3.3 (VI)
- new net BOOT0: R1.1, U1.36 (PA14)
- new net D+: J1.A6 (D+), J1.B6 (D+), U1.34 (PA10/PA12)
- new net D-: J1.A7 (D-), J1.B7 (D-), U1.33 (PA9/PA11)
- new net GND: C1.2, C2.2, C3.2, C4.2, C5.2, C6.2, C7.2, J1.A1 (GND), J1.A12 (GND), J1.B1 (GND), J1.B12 (GND), J1.S1 (SHIELD), R2.2, R3.2, SW1.2, SW2.1 (A), U1.7 (VSS), U2.2 (VN), U3.1 (GND)
- new net VBUS: F1.1, J1.A4 (VBUS), J1.A9 (VBUS), J1.B4 (VBUS), J1.B9 (VBUS)
- new net nRST: C5.1, SW1.1, U1.10 (PF2)
- no-connect marks 0 -> 2
Other:
- added sheet Switch Matrix (matrix.kicad_sch)

Commit message: Schematic initial completion
Parts:
- C1, C2, C3, C4, C5, C6, C7: footprint (none) -> Capacitor_SMD:C_0805_2012Metric
- F1: footprint (none) -> Fuse:Fuse_1206_3216Metric
- J1: footprint (none) -> Connector_USB:USB_C_Receptacle_HRO_TYPE-C-31-M-12
- R1, R2, R3: footprint (none) -> Resistor_SMD:R_0805_2012Metric
- SW1: footprint (none) -> Button_Switch_SMD:SW_SPST_TS-1088-xR020
- SW2: footprint (none) -> Button_Switch_SMD:SW_SPDT_PCM12
Changed lines of the file:
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@@
 			)
 		)
-		(property "Footprint" ""
+		(property "Footprint" "Connector_USB:USB_C_Receptacle_HRO_TYPE-C-31-M-12"
 			(at 153.67 73.66 0)
 			(effects
@@
 			)
 		)
-		(property "Footprint" ""
+		(property "Footprint" "Button_Switch_SMD:SW_SPST_TS-1088-xR020"
 			(at 149.86 31.75 0)
 			(effects
@@
 			)
 		)
-		(property "Footprint" ""
+		(property "Footprint" "Resistor_SMD:R_0805_2012Metric"
 			(at 194.31 33.528 90)
 			(effects
@@
 			)
 		)
-		(property "Footprint" ""
+		(property "Footprint" "Capacitor_SMD:C_0805_2012Metric"
 			(at 133.0452 34.29 0)
 			(effects
@@
 			)
 		)
-		(property "Footprint" ""
+		(property "Footprint" "Capacitor_SMD:C_0805_2012Metric"
 			(at 42.8752 38.1 0)
 			(effects
@@
 			)
 		)
-		(property "Footprint" ""
+		(property "Footprint" "Capacitor_SMD:C_0805_2012Metric"
 			(at 89.8652 34.29 0)
 			(effects
@@
 			)
 		)
-		(property "Footprint" ""
+		(property "Footprint" "Capacitor_SMD:C_0805_2012Metric"
 			(at 30.1752 38.1 0)
 			(effects
@@
 			)
 		)
-		(property "Footprint" ""
+		(property "Footprint" "Fuse:Fuse_1206_3216Metric"
 			(at 186.69 57.15 0)
 			(effects
@@
 			)
 		)
-		(property "Footprint" ""
+		(property "Footprint" "Capacitor_SMD:C_0805_2012Metric"
 			(at 102.5652 34.29 0)
 			(effects
@@
 			)
 		)
-		(property "Footprint" ""
+		(property "Footprint" "Capacitor_SMD:C_0805_2012Metric"
 			(at 205.4352 115.57 0)
 			(effects
@@
 			)
 		)
-		(property "Footprint" ""
+		(property "Footprint" "Resistor_SMD:R_0805_2012Metric"
 			(at 188.722 73.66 90)
 			(effects
@@
 			)
 		)
-		(property "Footprint" ""
+		(property "Footprint" "Resistor_SMD:R_0805_2012Metric"
 			(at 198.882 73.66 90)
 			(effects
@@
 			)
 		)
-		(property "Footprint" ""
+		(property "Footprint" "Capacitor_SMD:C_0805_2012Metric"
 			(at 180.0352 115.57 0)
 			(effects
@@
 			)
 		)
-		(property "Footprint" ""
+		(property "Footprint" "Button_Switch_SMD:SW_SPDT_PCM12"
 			(at 208.28 31.75 0)
 			(effects
